Commit message: cage einfuhren v0.3

File: gym_pybullet_drones/assets/cf2p.urdf (robot description, URDF)
Before this commit: robot cf2, 6 links, 5 joints
Links:
- added link magnet10_link, mass 0
- added link magnet11_link, mass 0
- added link magnet12_link, mass 0
- added link magnet13_link, mass 0
- added link magnet14_link, mass 0
- added link magnet15_link, mass 0
- added link magnet16_link, mass 0
- added link magnet1_link, mass 0
- added link magnet2_link, mass 0
- added link magnet3_link, mass 0
- added link magnet4_link, mass 0
- added link magnet5_link, mass 0
- added link magnet6_link, mass 0
- added link magnet7_link, mass 0
- added link magnet8_link, mass 0
- added link magnet9_link, mass 0
- link base_link: mass 0.027 -> 0.034; geometry collision box size=0.118 0.118 0.048; visual mesh filename=./cf2.dae scale=1 1 1
Joints:
- added joint magnet10_joint: type fixed, parent base_link, child magnet10_link
- added joint magnet11_joint: type fixed, parent base_link, child magnet11_link
- added joint magnet12_joint: type fixed, parent base_link, child magnet12_link
- added joint magnet13_joint: type fixed, parent base_link, child magnet13_link
- added joint magnet14_joint: type fixed, parent base_link, child magnet14_link
- added joint magnet15_joint: type fixed, parent base_link, child magnet15_link
- added joint magnet16_joint: type fixed, parent base_link, child magnet16_link
- added joint magnet1_joint: type fixed, parent base_link, child magnet1_link
- added joint magnet2_joint: type fixed, parent base_link, child magnet2_link
- added joint magnet3_joint: type fixed, parent base_link, child magnet3_link
- added joint magnet4_joint: type fixed, parent base_link, child magnet4_link
- added joint magnet5_joint: type fixed, parent base_link, child magnet5_link
- added joint magnet6_joint: type fixed, parent base_link, child magnet6_link
- added joint magnet7_joint: type fixed, parent base_link, child magnet7_link
- added joint magnet8_joint: type fixed, parent base_link, child magnet8_link
- added joint magnet9_joint: type fixed, parent base_link, child magnet9_link

Commit message: ppo v0.1

File: gym_pybullet_drones/assets/cf2p.urdf (robot description, URDF)
Before this commit: robot cf2, 22 links, 21 joints
Links:
- link base_link: geometry visual mesh filename=./cf2.dae scale=1 1 1
